Commit message: iiwa compiles, gato_pick&place_iiwa fails due to tuning/urdf issues

File: examples/iiwa-mpc/description/iiwa.urdf (robot description, URDF)
Before this commit: robot KUKAiiwa14, 10 links, 9 joints
Links:
- link L1: geometry collision mesh filename=iiwa_link_1.stl; visual mesh filename=iiwa_link_1.stl
- link L2: geometry collision mesh filename=iiwa_link_2.stl; visual mesh filename=iiwa_link_2.stl
- link L3: geometry collision mesh filename=iiwa_link_3.stl; visual mesh filename=iiwa_link_3.stl
- link L4: geometry collision mesh filename=iiwa_link_4.stl; visual mesh filename=iiwa_link_4.stl
- link L5: geometry collision mesh filename=iiwa_link_5.stl; visual mesh filename=iiwa_link_5.stl
- link L6: geometry collision mesh filename=iiwa_link_6.stl; visual mesh filename=iiwa_link_6.stl
- link L7: geometry collision mesh filename=iiwa_link_7.stl; visual mesh filename=iiwa_link_7.stl
- link contact: geometry 
- link iiwa_base: geometry collision mesh filename=iiwa_base.stl; visual mesh filename=iiwa_base.stl

Commit message: Validating solver with iiwa configuration

File: examples/iiwa-mpc/description/iiwa.urdf (robot description, URDF)
Before this commit: robot KUKAiiwa14, 10 links, 9 joints
Links:
- link contact: geometry collision sphere radius=0.033; visual sphere radius=0.033
