Commit message: update description

File: examples/iiwa_description/iiwa14.urdf (robot description, URDF)
Before this commit: robot iiwa14, 12 links, 11 joints
Links:
- removed link link_0
- removed link link_1
- removed link link_2
- removed link link_3
- removed link link_4
- removed link link_5
- removed link link_6
- removed link link_7
- removed link link_ee
- removed link link_ee_kuka
- removed link link_ee_kuka_mft_pneum
- added link L1, mass 3.94781; collision mesh filename=iiwa_link_1.stl; visual mesh filename=iiwa_link_1.stl
- added link L2, mass 4.50275; collision mesh filename=iiwa_link_2.stl; visual mesh filename=iiwa_link_2.stl
- added link L3, mass 2.45520; collision mesh filename=iiwa_link_3.stl; visual mesh filename=iiwa_link_3.stl
- added link L4, mass 2.61155; collision mesh filename=iiwa_link_4.stl; visual mesh filename=iiwa_link_4.stl
- added link L5, mass 3.41000; collision mesh filename=iiwa_link_5.stl; visual mesh filename=iiwa_link_5.stl
- added link L6, mass 3.38795; collision mesh filename=iiwa_link_6.stl; visual mesh filename=iiwa_link_6.stl
- added link L7, mass 0.35432; collision mesh filename=iiwa_link_7.stl; visual mesh filename=iiwa_link_7.stl
- added link contact, mass 0.057; collision sphere radius=0.033; visual sphere radius=0.033
- added link iiwa_base, mass 5; collision mesh filename=iiwa_base.stl; visual mesh filename=iiwa_base.stl
Joints:
- removed joint joint_0
- removed joint joint_1
- removed joint joint_2
- removed joint joint_3
- removed joint joint_4
- removed joint joint_5
- removed joint joint_6
- removed joint joint_ee
- removed joint joint_ee_kuka
- removed joint joint_ee_kuka_mft_pneum
- removed joint world_joint
- added joint A0: type fixed, parent world, child iiwa_base, origin xyz=0 0 0 rpy=0 0 0
- added joint A1: type revolute, parent iiwa_base, child L1, origin xyz=0.00000 0.00000 0.15750 rpy=0.0 0.0 0.0, axis 0 0 1, limit lower=-2.96706 upper=2.96706 effort=320 velocity=1.48353
- added joint A2: type revolute, parent L1, child L2, origin xyz=0.00000 0.00000 0.20250 rpy=2.3561944901923457 -1.5707962635746238 2.3561944901923457, axis 0 0 1, limit lower=-2.0944 upper=2.0944 effort=320 velocity=1.48353
- added joint A3: type revolute, parent L2, child L3, origin xyz=0.20450 0.00000 0.00000 rpy=1.5707963267948948 -4.371139000186238E-8 1.5707963705062866, axis 0 0 1, limit lower=-2.96706 upper=2.96706 effort=176 velocity=1.74533
- added joint A4: type revolute, parent L3, child L4, origin xyz=0.00000 0.00000 0.21550 rpy=1.5707963705062866 -0.0 0.0, axis 0 0 1, limit lower=-2.0944 upper=2.0944 effort=176 velocity=1.309
- added joint A5: type revolute, parent L4, child L5, origin xyz=0.00000 0.18450 0.00000 rpy=-1.5707963705062866 0.0 -0.0, axis 0 0 1, limit lower=-2.96706 upper=2.96706 effort=110 velocity=2.26893
- added joint A6: type revolute, parent L5, child L6, origin xyz=0.00000 -0.06070 0.21550 rpy=2.3561944901923457 -1.5707962635746238 2.3561944901923457, axis 0 0 1, limit lower=-2.0944 upper=2.0944 effort=40 velocity=2.35619
- added joint A7: type revolute, parent L6, child L7, origin xyz=0.08100 0.00000 0.06070 rpy=1.5707963267948948 -4.371139000186238E-8 1.5707963705062866, axis 0 0 1, limit lower=-3.05433 upper=3.05433 effort=40 velocity=2.35619
- added joint EE: type fixed, parent L7, child contact, origin xyz=0 0.0 0.04 rpy=0 0 0, limit lower=-10 upper=10 effort=1000 velocity=1000
